Commit message: fix namespaces

File: p_mcarvalho_description/urdf/p_mcarvalho.urdf.xacro (robot description, xacro)
@@ -142,5 +142,5 @@
     <parent link="base_link"/>
     <child link="base_scan"/>
-    <origin xyz="-0.064 0 0.122" rpy="0 0 0"/>
+    <origin xyz="-0.15 0 0.122" rpy="0 0 0"/>
   </joint>
   <link name="base_scan">
