Commit message: bumpers

File: p_mcarvalho_description/urdf/p_mcarvalho.gazebo.xacro (robot description, xacro)
@@ -6,4 +6,15 @@
   <xacro:arg name="imu_visual"    default="false"/>
   <gazebo reference="base_link">
+    <sensor name="base_link" type="contact">
+      <update_rate>1000.0</update_rate>
+      <always_on>true</always_on>
+      <contact>
+        <collision> "base_footprint_fixed_joint_lump__front_camera_link_collision_4" </collision>
+      </contact>
+      <plugin name="base_link_contact_sensor_plugin" filename="libgazebo_ros_bumper.so">
+        <bumperTopicName>contact</bumperTopicName>
+        <frameName>world</frameName>
+      </plugin>
+    </sensor>
     <!-- <material>Gazebo/DarkGrey</material> -->
     <material>Gazebo/${player_color}</material>

Commit message: bumpers

File: p_mcarvalho_description/urdf/p_mcarvalho.gazebo.xacro (robot description, xacro)
@@ -6,15 +6,4 @@
   <xacro:arg name="imu_visual"    default="false"/>
   <gazebo reference="base_link">
-    <sensor name="base_link" type="contact">
-      <update_rate>1000.0</update_rate>
-      <always_on>true</always_on>
-      <contact>
-        <collision> "base_footprint_fixed_joint_lump__front_camera_link_collision_4" </collision>
-      </contact>
-      <plugin name="base_link_contact_sensor_plugin" filename="libgazebo_ros_bumper.so">
-        <bumperTopicName>contact</bumperTopicName>
-        <frameName>world</frameName>
-      </plugin>
-    </sensor>
     <!-- <material>Gazebo/DarkGrey</material> -->
     <material>Gazebo/${player_color}</material>
@@ -212,3 +201,16 @@
     </sensor>
   </gazebo>
+  <gazebo reference="base_link">
+    <sensor name="base_link" type="contact">
+      <update_rate>1000.0</update_rate>
+      <always_on>true</always_on>
+      <contact>
+        <collision>base_footprint_fixed_joint_lump__base_link_collision</collision>
+      </contact>
+      <plugin name="base_link_contact_sensor_plugin" filename="libgazebo_ros_bumper.so">
+        <bumperTopicName>contact</bumperTopicName>
+        <frameName>world</frameName>
+      </plugin>
+    </sensor>
+  </gazebo>
 </robot>
